File: ergogen/output/pcbs/shield-pcb.kicad_pcb (KiCad board)
At the start: 2 copper layers, 118.1 x 90.8 mm, 26 parts

Commit message: ordered
Parts:
- removed _5: , MountingHole_2.2mm_M2_Pad_Via
- added _10: , MountingHole_2.2mm_M2_Pad_Via, F.Cu at (232.1, 155.5)
- moved _7 59.8 mm to (156.0, 129.6), turned to 5.33333 degrees
- moved _2 47.0 mm to (239.1, 100.5), turned to 0 degrees
- moved _9 35.6 mm to (212.1, 126.0)
- moved _6 18.0 mm to (154.3, 111.7)
- moved _8 17.0 mm to (212.1, 109.0)
- moved MCU 15.0 mm to (240.2, 132.5)
Connections:
- net B+ renamed RAW
- _2 pad 2: B- -> GND
Other:
- outline, holes or cut-outs redrawn
- board text added: "blog.imochoa.com"
