File: hardware/ergogen/output/pcbs/shield-pcb.kicad_pcb (KiCad board)
At the start: 2 copper layers, 115 x 93.8 mm, 25 parts

Commit message: feat: replace direct key inputs with diode matrix
Add a 5x4 diode matrix to each half and regenerate the PCB with 18 reversible SOD-123 footprints.

Update ZMK scanning and split transforms to match the matrix, reserve D21/AIN7 for battery sensing, and restore split battery reporting. Document the new pin map, diode orientation, and battery calibration requirements.
Parts:
- added D1: , ceoloide:diode_tht_sod123, F.Cu at (157.0, 150.0)
- added D10: , ceoloide:diode_tht_sod123, F.Cu at (211.0, 136.0)
- added D11: , ceoloide:diode_tht_sod123, F.Cu at (211.0, 119.0)
- added D12: , ceoloide:diode_tht_sod123, F.Cu at (211.0, 102.0)
- added D13: , ceoloide:diode_tht_sod123, F.Cu at (229.0, 138.9)
- added D14: , ceoloide:diode_tht_sod123, F.Cu at (229.0, 121.9)
- added D15: , ceoloide:diode_tht_sod123, F.Cu at (229.0, 104.9)
- added D16: , ceoloide:diode_tht_sod123, F.Cu at (202.0, 157.0)
- added D17: , ceoloide:diode_tht_sod123, F.Cu at (221.9, 161.4)
- added D18: , ceoloide:diode_tht_sod123, F.Cu at (239.9, 171.0)
- added D2: , ceoloide:diode_tht_sod123, F.Cu at (157.0, 133.0)
- added D3: , ceoloide:diode_tht_sod123, F.Cu at (157.0, 116.0)
- added D4: , ceoloide:diode_tht_sod123, F.Cu at (175.0, 136.0)
- added D5: , ceoloide:diode_tht_sod123, F.Cu at (175.0, 119.0)
- added D6: , ceoloide:diode_tht_sod123, F.Cu at (175.0, 102.0)
- added D7: , ceoloide:diode_tht_sod123, F.Cu at (193.0, 131.2)
- added D8: , ceoloide:diode_tht_sod123, F.Cu at (193.0, 114.2)
- added D9: , ceoloide:diode_tht_sod123, F.Cu at (193.0, 97.2)
Connections:
- MCU1 pad 10: thumb-zn_near_thumb -> col3
- MCU1 pad 11: thumb-zn_home_thumb -> P16
- MCU1 pad 12: thumb-zn_far_thumb -> P10
- MCU1 pad 123: grid-zn_ring_top -> P0
- MCU1 pad 124: grid-zn_middle_top -> P1
- MCU1 pad 13: grid-zn_inner_bottom -> P9
- MCU1 pad 14: grid-zn_index_bottom -> P8
- MCU1 pad 15: grid-zn_middle_bottom -> row3
- MCU1 pad 16: grid-zn_ring_bottom -> row2
- MCU1 pad 17: grid-zn_ring_home -> row1
- MCU1 pad 18: grid-zn_inner_home -> row0
- MCU1 pad 19: grid-zn_index_home -> P3
- MCU1 pad 20: grid-zn_middle_home -> P2
- MCU1 pad 5: grid-zn_inner_top -> P21
- MCU1 pad 6: grid-zn_index_top -> col2
- MCU1 pad 7: grid-zn_pinky_top -> col1
- MCU1 pad 8: grid-zn_pinky_home -> col0
- MCU1 pad 9: grid-zn_pinky_bottom -> col4
- S1 pad 2: GND -> col0
- S10 pad 2: GND -> col3
- S11 pad 2: GND -> col3
- S12 pad 2: GND -> col3
- S13 pad 2: GND -> col4
- S14 pad 2: GND -> col4
- S15 pad 2: GND -> col4
- S16 pad 2: GND -> col2
- S17 pad 2: GND -> col3
- S18 pad 2: GND -> col4
- S2 pad 2: GND -> col0
- S3 pad 2: GND -> col0
- S4 pad 2: GND -> col1
- S5 pad 2: GND -> col1
- S6 pad 2: GND -> col1
- S7 pad 2: GND -> col2
- S8 pad 2: GND -> col2
- S9 pad 2: GND -> col2
Routing:
- net row2: track 0.00 -> 12.0 mm, vias 0 -> 5
- net row1: track 0.00 -> 12.0 mm, vias 0 -> 5
- net row0: track 0.00 -> 12.0 mm, vias 0 -> 5
- net row3: track 0.00 -> 7.20 mm, vias 0 -> 3
- net thumb-zn_home_thumb: track 0.00 -> 2.40 mm, vias 0 -> 1
- net thumb-zn_far_thumb: track 0.00 -> 2.40 mm, vias 0 -> 1
- net thumb-zn_near_thumb: track 0.00 -> 2.40 mm, vias 0 -> 1
- net grid-zn_ring_top: track 0.00 -> 2.40 mm, vias 0 -> 1
- net grid-zn_ring_home: track 0.00 -> 2.40 mm, vias 0 -> 1
- net grid-zn_ring_bottom: track 0.00 -> 2.40 mm, vias 0 -> 1
- net grid-zn_pinky_top: track 0.00 -> 2.40 mm, vias 0 -> 1
- net grid-zn_pinky_home: track 0.00 -> 2.40 mm, vias 0 -> 1
- net grid-zn_pinky_bottom: track 0.00 -> 2.40 mm, vias 0 -> 1
- net grid-zn_middle_top: track 0.00 -> 2.40 mm, vias 0 -> 1
- net grid-zn_middle_home: track 0.00 -> 2.40 mm, vias 0 -> 1
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